File: H21R2/Design/H21R2.sch (EAGLE design)
At the start: 52 parts, among them IC1 ESP32-C3-MINI-1-N4, P1 HEXABIT_17.32_NO_P6_P7_P12, U1 STM32G0B1CEU6N, X1 8MHZ

Commit message: -Correct some documentation issues
Other:
- note added: "H21R2"
- note added: "H21R2_Backend"
- note added: "H21R2_Frontend"
- note removed: "H21R20"
- note removed: "H21R20_Backend"
- note removed: "H21R20_Frontend"
- note removed: "Ibrahim Zaeiter"
Changed lines of the file:
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@@
 <?xml version="1.0" encoding="utf-8"?>
 <!DOCTYPE eagle SYSTEM "eagle.dtd">
-<eagle version="9.6.2">
+<eagle version="9.6.1">
 <drawing>
 <settings>
@@
 <setting verticaltext="up"/>
 </settings>
-<grid distance="50" unitdist="mil" unit="mil" style="lines" multiple="1" display="yes" altdistance="0.01" altunitdist="inch" altunit="inch"/>
+<grid distance="0.1" unitdist="inch" unit="inch" style="lines" multiple="1" display="no" altdistance="0.01" altunitdist="inch" altunit="inch"/>
 <layers>
 <layer number="1" name="Top" color="4" fill="1" visible="no" active="no"/>
@@
 <text x="215.9" y="5.08" size="1.9304" layer="100" font="vector">Sheet   of</text>
 <text x="199.39" y="19.05" size="1.9304" layer="100" font="vector">Title</text>
-<text x="180.34" y="19.05" size="1.9304" layer="102" font="vector">H21R20</text>
+<text x="180.34" y="19.05" size="1.9304" layer="102" font="vector">H21R2</text>
 <text x="179.07" y="11.43" size="1.9304" layer="101" font="vector">ESP32-C3 Wifi+BLE</text>
-<text x="205.74" y="19.05" size="1.9304" layer="101" font="vector">H21R20_Backend</text>
+<text x="205.74" y="19.05" size="1.9304" layer="101" font="vector">H21R2_Backend</text>
 <wire x1="168.91" y1="3.81" x2="168.91" y2="8.128" width="0.1524" layer="205"/>
 <wire x1="168.91" y1="8.128" x2="168.91" y2="18.288" width="0.1524" layer="205"/>
@@
 <wire x1="231.14" y1="18.288" x2="231.14" y2="22.86" width="0.1524" layer="205"/>
 <text x="242.57" y="6.35" size="1.9304" layer="100" font="vector">www.hexabitz.com</text>
-<text x="180.34" y="5.08" size="1.9304" layer="101" font="vector">Ibrahim Zaeiter</text>
 <text x="204.47" y="83.82" size="1.778" layer="94">VDDIO2 Coupling</text>
 <text x="142.24" y="83.82" size="1.778" layer="94">VDD\\\VDDA Coupling</text>
@@
 <text x="215.9" y="5.08" size="1.9304" layer="100" font="vector">Sheet   of</text>
 <text x="199.39" y="20.32" size="1.9304" layer="100" font="vector">Title</text>
-<text x="180.34" y="20.32" size="1.9304" layer="102" font="vector">H21R20</text>
+<text x="180.34" y="20.32" size="1.9304" layer="102" font="vector">H21R2</text>
 <text x="179.07" y="11.43" size="1.9304" layer="101" font="vector">ESP32-C3 Wifi+BLE</text>
-<text x="205.74" y="20.32" size="1.9304" layer="101" font="vector">H21R20_Frontend</text>
+<text x="205.74" y="20.32" size="1.9304" layer="101" font="vector">H21R2_Frontend</text>
 <wire x1="168.75125" y1="4.1275" x2="168.75125" y2="8.4455" width="0.1524" layer="205"/>
 <wire x1="168.75125" y1="8.4455" x2="168.75125" y2="18.6055" width="0.1524" layer="205"/>
@@
 <wire x1="230.98125" y1="18.6055" x2="230.98125" y2="23.1775" width="0.1524" layer="205"/>
 <text x="242.57" y="6.35" size="1.9304" layer="100" font="vector">www.hexabitz.com</text>
-<text x="180.34" y="5.08" size="1.9304" layer="101" font="vector">Ibrahim Zaeiter</text>
 <text x="35.56" y="154.94" size="1.778" layer="102" align="center">To use external JTAG debugger
  desolder R11 &amp; R12 &amp; R13</text>
